Commit message: updates

File: dyros_bolt_description/robots/bolt10.urdf (robot description, URDF)
Before this commit: robot bolt10_urdf, 11 links, 10 joints
Links:
- link L_Foot: geometry collision box size=0.10 0.03 0.02; visual mesh filename=package://dyros_bolt_description/meshes/stl/L_Foot_box.stl
- link L_HipPitch_Link: geometry collision mesh filename=package://dyros_bolt_description/meshes/stl/L_HipPitch_Link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; visual mesh filename=package://dyros_bolt_description/meshes/stl/L_HipPitch_Link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
- link L_HipRoll_Link: geometry visual mesh filename=package://dyros_bolt_description/meshes/stl/L_HipRoll_Link.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
- link L_Lower_Leg: geometry collision mesh filename=package://dyros_bolt_description/meshes/stl/L_Lower_Leg.stl; visual mesh filename=package://dyros_bolt_description/meshes/stl/L_Lower_Leg.stl
- link L_Upper_Leg: geometry collision mesh filename=package://dyros_bolt_description/meshes/stl/L_Upper_Leg.stl; visual mesh filename=package://dyros_bolt_description/meshes/stl/L_Upper_Leg.stl
- link R_Foot: geometry collision box size=0.10 0.03 0.02; visual mesh filename=package://dyros_bolt_description/meshes/stl/R_Foot_box.stl
- link R_HipPitch_Link: geometry collision mesh filename=package://dyros_bolt_description/meshes/stl/R_HipPitch_Link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; visual mesh filename=package://dyros_bolt_description/meshes/stl/R_HipPitch_Link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
- link R_HipRoll_Link: geometry collision mesh filename=package://dyros_bolt_description/meshes/stl/R_HipRoll_Link.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; visual mesh filename=package://dyros_bolt_description/meshes/stl/R_HipRoll_Link.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
- link R_Lower_Leg: geometry collision mesh filename=package://dyros_bolt_description/meshes/stl/R_Lower_Leg.stl; visual mesh filename=package://dyros_bolt_description/meshes/stl/R_Lower_Leg.stl
- link R_Upper_Leg: geometry collision mesh filename=package://dyros_bolt_description/meshes/stl/R_Upper_Leg.stl; visual mesh filename=package://dyros_bolt_description/meshes/stl/R_Upper_Leg.stl
- link base_link: geometry collision sphere radius=0.15; visual mesh filename=package://dyros_bolt_description/meshes/stl/base_link.stl
